File: WiperModule/WiperModule.kicad_pcb (KiCad board)
At the start: 2 copper layers, 65.3 x 39.4 mm, 8 parts, among them J1 Conn_01x04, J2 Conn_01x04

Commit message: Updated to latest Kicad, images and added gitignore
Other:
- net class Default removed
